Commit message: add namespace for tf name

File: src/vehicle_simulator/urdf/camera.urdf.xacro (robot description, xacro)
@@ -1,4 +1,4 @@
 <robot xmlns:xacro="http://www.ros.org/wiki/xacro" name="example">
-  <link name="camera">
+  <link name="robot_0/camera">
     <collision>
       <origin xyz="0 0 0" rpy="0 0 0"/>
@@ -19,6 +19,6 @@
     </inertial>
   </link>
-  <gazebo reference="camera">
-    <sensor type="camera" name="camera">
+  <gazebo reference="robot_0/camera">
+    <sensor type="robot_0/camera" name="robot_0/camera">
       <update_rate>15.0</update_rate>
       <camera name="head">

File: src/vehicle_simulator/urdf/lidar.urdf.xacro (robot description, xacro)
@@ -1,7 +1,7 @@
 <?xml version="1.0"?>
 <robot xmlns:xacro="http://www.ros.org/wiki/xacro" name="example">
-  <link name="lidar" />
+  <link name="robot_0/lidar" />
   <xacro:include filename="$(find velodyne_description)/urdf/VLP-16.urdf.xacro"/>
-  <xacro:VLP-16 parent="lidar" name="velodyne" topic="velodyne_points" hz="6.3" samples="350" min_range="0.1">
+  <xacro:VLP-16 parent="robot_0/lidar" name="velodyne" topic="velodyne_points" hz="6.3" samples="350" min_range="0.1">
     <origin xyz="0 0 0" rpy="0 0 0" />
   </xacro:VLP-16>
